Commit message: add diff_drive_controller

File: src/mbot_description_gazebo/urdf/mbot_base_gazebo.xacro (robot description, xacro)
@@ -88,5 +88,5 @@
         </link>
         <gazebo reference="${prefix}_wheel_link">
-            <material>Gazebo/Gray</material>
+            <material>Gazebo/Black</material>
         </gazebo>
         <!-- Transmission is important to link the joints and the controller -->
@@ -172,10 +172,10 @@
         <caster prefix="back"  reflect="1"/>
         <!-- controller -->
-        <gazebo>
+        <!--<gazebo>
             <plugin name="differential_drive_controller"
                     filename="libgazebo_ros_diff_drive.so">
                 <rosDebugLevel>Debug</rosDebugLevel>
                 <publishWheelTF>true</publishWheelTF>
-                <robotNamespace>/</robotNamespace>
+                <robotNamespace>/mbot</robotNamespace>
                 <publishTf>1</publishTf>
                 <publishWheelJointState>true</publishWheelJointState>
@@ -195,4 +195,11 @@
                 <robotBaseFrame>base_footprint</robotBaseFrame>
             </plugin>
+        </gazebo> -->
+        <gazebo>
+            <plugin name="gazebo_ros_control" filename="libgazebo_ros_control.so">
+                <robotNamespace>/mbot</robotNamespace>
+                <robotSimType>gazebo_ros_control/DefaultRobotHWSim</robotSimType>
+                <legacyModeNS>true</legacyModeNS>
+             </plugin>
         </gazebo>
     </xacro:macro>

File: src/pick_ball_mbot/urdf/pick_ball_mbot.urdf (robot description, URDF)
Before this commit: robot pick_ball_mbot, 11 links, 10 joints
Links:
- removed link front_wheel
- removed link middle_transport
- removed link rear_collector
- removed link right_wheel
- added link front_left_wheel, mass 0.0937829390237727; collision mesh filename=package://pick_ball_mbot/meshes/front_left_wheel.STL; visual mesh filename=package://pick_ball_mbot/meshes/front_left_wheel.STL
- added link front_right_wheel, mass 0.0937829390237727; collision mesh filename=package://pick_ball_mbot/meshes/front_right_wheel.STL; visual mesh filename=package://pick_ball_mbot/meshes/front_right_wheel.STL
- added link rear_left_wheel, mass 0.0937829390237727; collision mesh filename=package://pick_ball_mbot/meshes/rear_left_wheel.STL; visual mesh filename=package://pick_ball_mbot/meshes/rear_left_wheel.STL
- added link rear_right_wheel, mass 0.0937829390237727; collision mesh filename=package://pick_ball_mbot/meshes/rear_right_wheel.STL; visual mesh filename=package://pick_ball_mbot/meshes/rear_right_wheel.STL
- link base_link: mass 1.05139109376071 -> 1.0824
- link collector: mass 0.192616334199706 -> 0.373810739586063
- link left_cover: mass 0.348968668389308 -> 0.348968668389245
- link left_support_rod: mass 0.00511240249563706 -> 0.00511240249562874
- link paddle: mass 0.16555 -> 0
- link right_support_rod: mass 0.00511240249563707 -> 0.00511240249562874
Joints:
- removed joint front_wheel_joint
- removed joint middle_transport_joint
- removed joint rear_collector_joint
- removed joint right_wheel_joint
- added joint front_left_wheel_joint: type continuous, parent base_link, child front_left_wheel, origin xyz=0.12101 -0.10059 -0.030048 rpy=1.5708 0.24454 -1.546, axis 0 0 0
- added joint front_right_wheel_joint: type continuous, parent base_link, child front_right_wheel, origin xyz=-0.066074 -0.10152 -0.030048 rpy=1.5708 1.5309 -1.5744, axis 0 0 0
- added joint rear_left_wheel_joint: type continuous, parent base_link, child rear_left_wheel, origin xyz=0.092074 -0.24356 -0.030048 rpy=1.5708 0 -1.5708, axis 0 0 0
- added joint rear_right_wheel_joint: type continuous, parent base_link, child rear_right_wheel, origin xyz=-0.095123 -0.24365 -0.030048 rpy=-1.5708 1.3457 -1.5685, axis 0 0 0
- joint collector_joint: origin xyz=-0.0073431 -0.4104 -0.061965 rpy=-1.5708 0 -1.5708 -> xyz=0.0094753 -0.11331 0.048119 rpy=1.5708 0 0
- joint left_cover_joint: origin xyz=-0.00070327 -0.2264 -0.072965 rpy=0 0 0 -> xyz=0.01014 -0.11017 0.072246 rpy=-1.5708 0 0; parent base_link -> collector
- joint left_support_rod_joint: origin xyz=0.024614 -0.15428 -0.057965 rpy=1.5708 0 3.1416 -> xyz=0.044933 -0.11344 -0.047048 rpy=1.5708 0 3.1416
- joint paddle_joint: origin xyz=0 -0.0023183 0.047035 rpy=-2.3269 0 3.1416 -> xyz=0 0.038521 0.057952 rpy=2.6432 0 -3.1416
- joint right_cover_joint: origin xyz=-0.065843 -0.0023183 0.047035 rpy=3.1416 -1.5708 0 -> xyz=-0.055 0.0098333 -0.15183 rpy=-1.5708 0 1.5708; parent base_link -> collector
- joint right_support_rod_joint: origin xyz=-0.0392756380929201 -0.154282545794808 -0.0579653445088367 rpy=1.5707963267949 0 0 -> xyz=-0.018957 -0.11344 -0.047048 rpy=1.5708 0 0

File: src/pick_ball_mbot/urdf/pick_ball_mbot_base_gazebo.xacro (robot description, xacro)
@@ -1,31 +1,7 @@
 <?xml version="1.0"?>
 <robot name="pick_ball_mbot" xmlns:xacro="http://www.ros.org/wiki/xacro">
-    <xacro:property name="wheel_mass"   value="2" />
-    <xacro:property name="wheel_radius" value="0.06"/>
-    <xacro:property name="wheel_length" value="0.025"/>
-    <xacro:property name="wheel_joint_y" value="0.19"/>
-    <xacro:property name="wheel_joint_z" value="0.05"/>
-    <!-- Defining the colors used in this robot -->
-    <material name="yellow">
-        <color rgba="1 0.4 0 1"/>
-    </material>
-    <material name="black">
-        <color rgba="0 0 0 0.95"/>
-    </material>
-    <material name="gray">
-        <color rgba="0.75 0.75 0.75 1"/>
-    </material>
-    <xacro:macro name="joint_trans"  params="joint_name">
-        <transmission name="${joint_name}_trans">
-            <type>transmission_interface/SimpleTransmission</type>
-            <joint name="${joint_name}" >
-                <hardwareInterface>hardware_interface/VelocityJointInterface</hardwareInterface>
-            </joint>
-            <actuator name="${joint_name}_motor">
-                <hardwareInterface>hardware_interface/VelocityJointInterface</hardwareInterface>
-                <mechanicalReduction>1</mechanicalReduction>
-            </actuator>
-        </transmission>
-    </xacro:macro>
+    <xacro:property name="collector_mass_multiplier" value="15"/>
+    <xacro:property name="base_link_mass_multiplier" value="8"/>
+    <xacro:property name="cover_mass_multiplier" value="1"/>
     <xacro:macro name="pick_ball_mbot_base_gazebo">
         <origin xyz="1 1 1" rpy="0 0 0" />
@@ -46,19 +22,19 @@
             <child link="base_link" />
         </joint>
-        <link
+         <link
             name="base_link">
             <inertial>
             <origin
-                xyz="-0.0073430681844793 -0.0240899963415031 0.216409188578357"
-                rpy="0 0 0" />
-            <mass
-                value="1.05139109376071" />
-            <inertia
-                ixx="0.00348499733987661"
-                ixy="5.59664608948403E-21"
-                ixz="-8.26305565804843E-20"
-                iyy="0.00365982960162949"
-                iyz="-0.000149638202350733"
-                izz="0.00152216475016813" />
+                xyz="0.012976 -0.013657 0.17563"
+                rpy="0 0 0" />
+            <mass
+                value="1.0824" />
+            <inertia
+                ixx="${base_link_mass_multiplier*0.0036507}"
+                ixy="${base_link_mass_multiplier*(5.8245E-21)}"
+                ixz="${base_link_mass_multiplier*(-1.7168E-19)}"
+                iyy="${base_link_mass_multiplier*0.0038702}"
+                iyz="${base_link_mass_multiplier*(-0.00014855)}"
+                izz="${base_link_mass_multiplier*0.0015847}" />
             </inertial>
             <visual>
@@ -73,5 +49,5 @@
                 name="">
                 <color
-                rgba="0.686274509803922 0 0 1" />
+                rgba="0.79216 0.81961 0.93333 1" />
             </material>
             </visual>
@@ -87,18 +63,283 @@
         </link>
         <link
+            name="front_right_wheel">
+            <inertial>
+            <origin
+                xyz="3.2106E-12 -1.2799E-13 0.014176"
+                rpy="0 0 0" />
+            <mass
+                value="0.093783" />
+            <inertia
+                ixx="3.0977E-05"
+                ixy="1.1309E-09"
+                ixz="6.3388E-15"
+                iyy="3.1005E-05"
+                iyz="-2.5278E-16"
+                izz="4.7784E-05" />
+            </inertial>
+            <visual>
+            <origin
+                xyz="0 0 0"
+                rpy="0 0 0" />
+            <geometry>
+                <mesh
+                filename="package://pick_ball_mbot/meshes/front_right_wheel.STL" />
+            </geometry>
+            <material
+                name="">
+                <color
+                rgba="1 1 1 1" />
+            </material>
+            </visual>
+            <collision>
+            <origin
+                xyz="0 0 0"
+                rpy="0 0 0" />
+            <geometry>
+                <mesh
+                filename="package://pick_ball_mbot/meshes/front_right_wheel.STL" />
+            </geometry>
+            </collision>
+        </link>
+        <joint
+            name="front_right_wheel_joint"
+            type="continuous">
+            <origin
+            xyz="-0.066074 -0.10152 -0.030048"
+            rpy="1.5708 1.5309 -1.5744" />
+            <parent
+            link="base_link" />
+            <child
+            link="front_right_wheel" />
+            <axis
+            xyz="0 0 0" />
+        </joint>
+        <link
+            name="front_left_wheel">
+            <inertial>
+            <origin
+                xyz="7.3687E-13 -3.129E-12 0.014824"
+                rpy="0 0 0" />
+            <mass
+                value="0.093783" />
+            <inertia
+                ixx="3.1004E-05"
+                ixy="6.672E-09"
+                ixz="-1.5055E-15"
+                iyy="3.0979E-05"
+                iyz="6.1608E-15"
+                izz="4.7784E-05" />
+            </inertial>
+            <visual>
+            <origin
+                xyz="0 0 0"
+                rpy="0 0 0" />
+            <geometry>
+                <mesh
+                filename="package://pick_ball_mbot/meshes/front_left_wheel.STL" />
+            </geometry>
+            <material
+                name="">
+                <color
+                rgba="1 1 1 1" />
+            </material>
+            </visual>
+            <collision>
+            <origin
+                xyz="0 0 0"
+                rpy="0 0 0" />
+            <geometry>
+                <mesh
+                filename="package://pick_ball_mbot/meshes/front_left_wheel.STL" />
+            </geometry>
+            </collision>
+        </link>
+        <joint
+            name="front_left_wheel_joint"
+            type="continuous">
+            <origin
+            xyz="0.12101 -0.10059 -0.030048"
+            rpy="1.5708 0.24454 -1.546" />
+            <parent
+            link="base_link" />
+            <child
+            link="front_left_wheel" />
+            <axis
+            xyz="0 0 0" />
+        </joint>
+        <link
+            name="rear_left_wheel">
+            <inertial>
+            <origin
+                xyz="-2.77555756156289E-17 3.21316931395366E-12 -0.0141764123448539"
+                rpy="0 0 0" />
+            <mass
+                value="0.0937829390237727" />
+            <inertia
+                ixx="3.10055399070393E-05"
+                ixy="-2.36350053451677E-24"
+                ixz="5.92798954623863E-20"
+                iyy="3.09771368078223E-05"
+                iyz="-6.34439778292892E-15"
+                izz="4.77838078287253E-05" />
+            </inertial>
+            <visual>
+            <origin
+                xyz="0 0 0"
+                rpy="0 0 0" />
+            <geometry>
+                <mesh
+                filename="package://pick_ball_mbot/meshes/rear_left_wheel.STL" />
+            </geometry>
+            <material
+                name="">
+                <color
+                rgba="1 1 1 1" />
+            </material>
+            </visual>
+            <collision>
+            <origin
+                xyz="0 0 0"
+                rpy="0 0 0" />
+            <geometry>
+                <mesh
+                filename="package://pick_ball_mbot/meshes/rear_left_wheel.STL" />
+            </geometry>
+            </collision>
+        </link>
+        <joint
+            name="rear_left_wheel_joint"
+            type="continuous">
+            <origin
+            xyz="0.092074 -0.24356 -0.030048"
+            rpy="1.5708 0 -1.5708" />
+            <parent
+            link="base_link" />
+            <child
+            link="rear_left_wheel" />
+            <axis
+            xyz="0 0 0" />
+        </joint>
+        <link
+            name="rear_right_wheel">
+            <inertial>
+            <origin
+                xyz="3.1321E-12 7.1729E-13 0.014824"
+                rpy="0 0 0" />
+            <mass
+                value="0.093783" />
+            <inertia
+                ixx="3.0979E-05"
+                ixy="-6.1803E-09"
+                ixz="-6.184E-15"
+                iyy="3.1004E-05"
+                iyz="-1.4162E-15"
+                izz="4.7784E-05" />
+            </inertial>
+            <visual>
+            <origin
+                xyz="0 0 0"
+                rpy="0 0 0" />
+            <geometry>
+                <mesh
+                filename="package://pick_ball_mbot/meshes/rear_right_wheel.STL" />
+            </geometry>
+            <material
+                name="">
+                <color
+                rgba="1 1 1 1" />
+            </material>
+            </visual>
+            <collision>
+            <origin
+                xyz="0 0 0"
+                rpy="0 0 0" />
+            <geometry>
+                <mesh
+                filename="package://pick_ball_mbot/meshes/rear_right_wheel.STL" />
+            </geometry>
+            </collision>
+        </link>
+        <joint
+            name="rear_right_wheel_joint"
+            type="continuous">
+            <origin
+            xyz="-0.095123 -0.24365 -0.030048"
+            rpy="-1.5708 1.3457 -1.5685" />
+            <parent
+            link="base_link" />
+            <child
+            link="rear_right_wheel" />
+            <axis
+            xyz="0 0 0" />
+        </joint>
+        <link
+            name="collector">
+            <inertial>
+            <origin
+                xyz="0.0029090749423291 -0.040890215457459 0.173468819063092"
+                rpy="0 0 0" />
+            <mass
+                value="${collector_mass_multiplier*(0.373)}" />
+            <inertia
+                ixx="${collector_mass_multiplier*(0.003466)}"
+                ixy="${collector_mass_multiplier*(9.698529E-06)}"
+                ixz="${collector_mass_multiplier*(-2.849826E-05)}"
+                iyy="${collector_mass_multiplier*(0.0042937)}"
+                iyz="${collector_mass_multiplier*(0.0005667)}"
+                izz="${collector_mass_multiplier*(0.0019856)}" />
+            </inertial>
+            <visual>
+            <origin
+                xyz="0 0 0"
+                rpy="0 0 0" />
+            <geometry>
+                <mesh
+                filename="package://pick_ball_mbot/meshes/collector.STL" />
+            </geometry>
+            <material
+                name="">
+                <color
+                rgba="0.792156862745098 0.819607843137255 0.933333333333333 1" />
+            </material>
+            </visual>
+            <collision>
+            <origin
+                xyz="0 0 0"
+                rpy="0 0 0" />
+            <geometry>
+                <mesh
+                filename="package://pick_ball_mbot/meshes/collector.STL" />
+            </geometry>
+            </collision>
+        </link>
+        <joint
+            name="collector_joint"
+            type="fixed">
+            <origin
+            xyz="0.0094753 -0.11331 0.048119"
+            rpy="1.5708 0 0" />
+            <parent
+            link="base_link" />
+            <child
+            link="collector" />
+            <axis
+            xyz="0 0 0" />
+        </joint>
+        <link
             name="left_cover">
             <inertial>
             <origin
-                xyz="0.0339621470957772 0.172876722995914 0.102900925287299"
-                rpy="0 0 0" />
-            <mass
-                value="0.348968668389308" />
-            <inertia
-                ixx="0.00220864018472111"
-                ixy="-9.94750925639056E-05"
-                ixz="-0.000119883170893649"
-                iyy="0.00198390619787086"
-                iyz="-0.000357322467893291"
-                izz="0.000935622380947324" />
+                xyz="0.0339621470957824 0.172876722995866 0.102900925287308"
+                rpy="0 0 0" />
+            <mass
+                value="0.348968668389245" />
+            <inertia
+                ixx="0.00220864016861759"
+                ixy="-9.94750925638527E-05"
+                ixz="-0.000119883170893584"
+                iyy="0.00198390619746038"
+                iyz="-0.000357322467893688"
+                izz="0.000935622364254192" />
             </inertial>
             <visual>
@@ -130,8 +371,8 @@
             type="fixed">
             <origin
-            xyz="-0.00070327 -0.2264 -0.072965"
-            rpy="0 0 0" />
-            <parent
-            link="base_link" />
+            xyz="0.01014 -0.11017 0.072246"
+            rpy="-1.5708 0 0" />
+            <parent
+            link="collector" />
             <child
             link="left_cover" />
@@ -140,17 +381,73 @@
         </joint>
         <link
+            name="paddle">
+            <inertial>
+            <origin
+                xyz="0.00973380728811933 3.27377014386343E-14 -8.10081168811649E-13"
+                rpy="0 0 0" />
+            <mass
+                value="0.165548548604918" />
+            <inertia
+                ixx="0.000631829797905281"
+                ixy="-1.39557756740262E-16"
+                ixz="-5.34445213789333E-15"
+                iyy="0.00050636909780647"
+                iyz="-5.81383519885487E-13"
+                izz="0.000506369100143511" />
+            </inertial>
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
File: src/pick_ball_mbot/urdf/pick_ball_mbot_gazebo.xacro (robot description, xacro)
@@ -3,3 +3,63 @@
     <xacro:include filename="$(find pick_ball_mbot)/urdf/pick_ball_mbot_base_gazebo.xacro" />
     <pick_ball_mbot_base_gazebo/>
+    <xacro:macro name="joint_trans"  params="joint_name">
+        <transmission name="${joint_name}_trans">
+            <type>transmission_interface/SimpleTransmission</type>
+            <joint name="${joint_name}" >
+                <hardwareInterface>hardware_interface/VelocityJointInterface</hardwareInterface>
+            </joint>
+            <actuator name="${joint_name}_motor">
+                <hardwareInterface>hardware_interface/VelocityJointInterface</hardwareInterface>
+                <mechanicalReduction>1</mechanicalReduction>
+            </actuator>
+        </transmission>
+    </xacro:macro>
+    <!--- design color for mbot -->
+    <gazebo reference="left_cover">
+        <material>Gazebo/Red</material>
+    </gazebo>
+    <gazebo reference="right_cover">
+        <material>Gazebo/Red</material>
+    </gazebo>
+    <gazebo reference="base_link">
+        <material>Gazebo/Blue</material>
+    </gazebo>
+    <gazebo reference="front_right_wheel">
+        <material>Gazebo/Black</material>
+    </gazebo>
+    <gazebo reference="front_left_wheel">
+        <material>Gazebo/Black</material>
+    </gazebo>
+    <gazebo reference="rear_right_wheel">
+        <material>Gazebo/Black</material>
+    </gazebo>
+    <gazebo reference="rear_left_wheel">
+        <material>Gazebo/Black</material>
+    </gazebo>
+    <gazebo reference="collector">
+        <material>Gazebo/Wood</material>
+    </gazebo>
+    <gazebo reference="paddle">
+        <material>Gazebo/Black</material>
+    </gazebo>
+    <gazebo reference="right_support_rod">
+        <material>Gazebo/Purple</material>
+    </gazebo>
+        <gazebo reference="left_support_rod">
+        <material>Gazebo/Purple</material>
+    </gazebo>
+    <!-- design transmission for joint-->
+    <joint_trans joint_name="front_right_wheel_joint"/>
+    <joint_trans joint_name="front_left_wheel_joint"/>
+    <joint_trans joint_name="rear_right_wheel_joint"/>
+    <joint_trans joint_name="rear_left_wheel_joint"/>
+    <joint_trans joint_name="paddle_joint"/>
+    <!-- design controller for joint-->
+    <gazebo>
+        <plugin name="gazebo_ros_control" filename="libgazebo_ros_control.so">
+            <robotNamespace>/pick_ball_mbot</robotNamespace>
+            <robotSimType>gazebo_ros_control/DefaultRobotHWSim</robotSimType>
+            <legacyModeNS>true</legacyModeNS>
+            </plugin>
+    </gazebo>
 </robot>

Commit message: adjust the params of HoughCircle, better recognition performace

File: src/mbot_description_gazebo/urdf/mbot_base_gazebo.xacro (robot description, xacro)
@@ -147,23 +147,4 @@
             <child link="base_link" />
         </joint>
-        <!--<link name="base_link">
-            <visual>
-                <origin xyz=" 0 0 0" rpy="0 0 0" />
-                <geometry>
-                    <cylinder length="${base_length}" radius="${base_radius}"/>
-                </geometry>
-                <material name="yellow" />
-            </visual>
-            <collision>
-                <origin xyz=" 0 0 0" rpy="0 0 0" />
-                <geometry>
-                    <cylinder length="${base_length}" radius="${base_radius}"/>
-                </geometry>
-            </collision>
-            <cylinder_inertial_matrix  m="${base_mass}" r="${base_radius}" h="${base_length}" />
-        </link>
-        <gazebo reference="base_link">
-            <material>Gazebo/Blue</material>
-        </gazebo>-->
         <base_link/>
         <wheel prefix="left"  reflect="-1"/>
