Commit message: use skid_steer_drive_controller to control a car which have four wheels, adjust the angle of kinect, add extend board to pick_ball_mbot_description

File: src/mbot/mbot_description_gazebo/urdf/sensors/lidar_gazebo.xacro (robot description, xacro)
@@ -38,6 +38,8 @@
                         <samples>360</samples>
                         <resolution>1</resolution>
-                        <min_angle>-3</min_angle>
-                        <max_angle>3</max_angle>
+                        <!--<min_angle>-3</min_angle>
+                        <max_angle>3</max_angle>-->
+                        <min_angle>0.0</min_angle>
+                        <max_angle>6.28319</max_angle>
                       </horizontal>
                     </scan>

File: src/pick_ball_mbot/pick_ball_mbot_description/urdf/pick_ball_mbot_base.xacro (robot description, xacro)
@@ -2,7 +2,8 @@
 <robot name="pick_ball_mbot_description" xmlns:xacro="http://www.ros.org/wiki/xacro">
     <xacro:property name="M_PI" value="3.1415926"/>
-    <xacro:property name="collector_mass_multiplier" value="15"/>
-    <xacro:property name="base_link_mass_multiplier" value="8"/>
-    <xacro:property name="cover_mass_multiplier" value="1"/>
+    <xacro:property name="collector_mass_multiplier" value="2"/>
+    <xacro:property name="base_link_mass_multiplier" value="2"/>
+    <xacro:property name="cover_mass_multiplier" value="2"/>
+    <xacro:property name="wheel_mass_multiplier" value="2"/>
     <xacro:macro name="pick_ball_mbot_base_gazebo">
         <link name="base_footprint">
@@ -69,12 +70,12 @@
             rpy="0 0 0" />
         <mass
-            value="0.093783" />
-        <inertia
-            ixx="3.0979E-05"
-            ixy="-6.7569E-09"
-            ixz="-6.6396E-15"
-            iyy="3.1004E-05"
-            iyz="-1.6704E-15"
-            izz="4.7784E-05" />
+            value="${wheel_mass_multiplier*0.093783}" />
+        <inertia
+            ixx="${wheel_mass_multiplier*(3.0979E-05)}"
+            ixy="${wheel_mass_multiplier*(-6.7569E-09)}"
+            ixz="${wheel_mass_multiplier*(-6.6396E-15)}"
+            iyy="${wheel_mass_multiplier*(3.1004E-05)}"
+            iyz="${wheel_mass_multiplier*(-1.6704E-15)}"
+            izz="${wheel_mass_multiplier*(4.7784E-05)}" />
         </inertial>
         <visual>
@@ -122,12 +123,12 @@
             rpy="0 0 0" />
         <mass
-            value="0.093783" />
-        <inertia
-            ixx="3.0978E-05"
-            ixy="-3.4152E-09"
-            ixz="-6.7962E-15"
-            iyy="3.1005E-05"
-            iyz="-8.2473E-16"
-            izz="4.7784E-05" />
+            value="${wheel_mass_multiplier*0.093783}" />
+        <inertia
+            ixx="${wheel_mass_multiplier*(3.0978E-05)}"
+            ixy="${wheel_mass_multiplier*(-3.4152E-09)}"
+            ixz="${wheel_mass_multiplier*(-6.7962E-15)}"
+            iyy="${wheel_mass_multiplier*(3.1005E-05)}"
+            iyz="${wheel_mass_multiplier*(-8.2473E-16)}"
+            izz="${wheel_mass_multiplier*(4.7784E-05)}" />
         </inertial>
         <visual>
@@ -175,12 +176,12 @@
             rpy="0 0 0" />
         <mass
-            value="0.0937829390237726" />
-        <inertia
-            ixx="3.10054780216612E-05"
-            ixy="1.32435143883117E-09"
-            ixz="2.9614191177372E-16"
-            iyy="3.09771986932004E-05"
-            iyz="-6.33701481449748E-15"
-            izz="4.77838078287252E-05" />
+            value="${wheel_mass_multiplier*0.093783}" />
+        <inertia
+            ixx="${wheel_mass_multiplier*(3.10054780216612E-05)}"
+            ixy="${wheel_mass_multiplier*(1.32435143883117E-09)}"
+            ixz="${wheel_mass_multiplier*(2.9614191177372E-16)}"
+            iyy="${wheel_mass_multiplier*(3.09771986932004E-05)}"
+            iyz="${wheel_mass_multiplier*(-6.33701481449748E-15)}"
+            izz="${wheel_mass_multiplier*(4.77838078287252E-05)}" />
         </inertial>
         <visual>
@@ -228,12 +229,12 @@
             rpy="0 0 0" />
         <mass
-            value="0.0937829390237727" />
-        <inertia
-            ixx="3.09771374888205E-05"
-            ixy="1.39076431308829E-10"
-            ixz="6.3436675045065E-15"
-            iyy="3.10055392260229E-05"
-            iyz="-2.99974052448107E-17"
-            izz="4.77838078287253E-05" />
+            value="${wheel_mass_multiplier*0.093783}" />
+        <inertia
+            ixx="${wheel_mass_multiplier*(3.09771374888205E-05)}"
+            ixy="${wheel_mass_multiplier*(1.39076431308829E-10)}"
+            ixz="${wheel_mass_multiplier*(6.3436675045065E-15)}"
+            iyy="${wheel_mass_multiplier*(3.10055392260229E-05)}"
+            iyz="${wheel_mass_multiplier*(-2.99974052448107E-17)}"
+            izz="${wheel_mass_multiplier*(4.77838078287253E-05)}" />
         </inertial>
         <visual>
@@ -334,12 +335,12 @@
             rpy="0 0 0" />
         <mass
-            value="0.35719" />
-        <inertia
-            ixx="0.0023208"
-            ixy="-0.00015274"
-            ixz="-8.1174E-05"
-            iyy="0.0020745"
-            iyz="-0.00030739"
-            izz="0.0010449" />
+            value="${cover_mass_multiplier*(0.35719)}" />
+        <inertia
+            ixx="${cover_mass_multiplier*(0.0023208)}"
+            ixy="${cover_mass_multiplier*(-0.00015274)}"
+            ixz="${cover_mass_multiplier*(-8.1174E-05)}"
+            iyy="${cover_mass_multiplier*(0.0020745)}"
+            iyz="${cover_mass_multiplier*(-0.00030739)}"
+            izz="${cover_mass_multiplier*(0.0010449)}" />
         </inertial>
         <visual>
@@ -387,12 +388,12 @@
             rpy="0 0 0" />
         <mass
-            value="0.11834" />
-        <inertia
-            ixx="0.00023044"
-            ixy="-3.8219E-06"
-            ixz="2.9166E-05"
-            iyy="0.00047003"
-            iyz="-3.578E-05"
-            izz="0.00064825" />
+            value="${cover_mass_multiplier*(0.11834)}" />
+        <inertia
+            ixx="${cover_mass_multiplier*(0.00023044)}"
+            ixy="${cover_mass_multiplier*(-3.8219E-06)}"
+            ixz="${cover_mass_multiplier*(2.9166E-05)}"
+            iyy="${cover_mass_multiplier*(0.00047003)}"
+            iyz="${cover_mass_multiplier*(-3.578E-05)}"
+            izz="${cover_mass_multiplier*(0.00064825)}" />
         </inertial>
         <visual>

File: src/pick_ball_mbot/pick_ball_mbot_description/urdf/pick_ball_mbot_gazebo.xacro (robot description, xacro)
@@ -6,17 +6,33 @@
     <xacro:include filename="$(find pick_ball_mbot_description)/urdf/joint_transmission_gazebo.xacro" />
     <xacro:include filename="$(find pick_ball_mbot_description)/urdf/paddle_gazebo.xacro" />
-    <xacro:property name="wheel_mu" value="3"/>
-        <!-- kinect -->
+    <xacro:include filename="$(find pick_ball_mbot_description)/urdf/extend_board.xacro" />
+    <xacro:include filename="$(find pick_ball_mbot_description)/urdf/top_stage_gazebo.xacro" />
+    <xacro:property name="wheel_mu1" value="10"/>
+    <xacro:property name="wheel_mu2" value="50"/>
+    <!-- extend board -->
+    <joint name="extend_board_joint" type="fixed">
+        <origin xyz="-0.0050 0.295 0.238" rpy="0 0 1.5707" />
+        <parent link="left_cover"/>
+        <child link="extend_board"/>
+    </joint>
+    <extend_board/>
+    <!-- kinect -->
     <joint name="kinect_joint" type="fixed">
-        <!--<origin xyz="-0.00214019 0.22491813 0.25000000" rpy="1.57079028 0 3.14159265" />-->
-        <origin xyz="-0.0050 0.2250 0.251" rpy="0 0 1.5707" />
-        <parent link="left_cover"/>
+        <origin xyz="0.05 0 0.01" rpy="0 0.55 0" />
+        <parent link="extend_board"/>
         <child link="kinect_link"/>
     </joint>
     <xacro:kinect_camera prefix="kinect"/>
+    <!-- top_stage -->
+    <joint name="top_stage_joint" type="fixed">
+        <origin xyz="0.015 0 0.015" rpy="0 0 0" />
+        <parent link="extend_board"/>
+        <child link="top_stage_link"/>
+    </joint>
+    <xacro:top_stage_link />
     <!-- lidar -->
     <joint name="lidar_joint" type="fixed">
-        <origin xyz="0 0 0.030" rpy="0 0 0" />
-        <parent link="kinect_link"/>
+        <origin xyz="0 0 0.02" rpy="0 0 0" />
+        <parent link="top_stage_link"/>
         <child link="laser_link"/>
     </joint>
@@ -63,56 +79,44 @@
     </gazebo>
     <!-- friction -->
-    <gazebo reference="front_left_wheel">
-        <mu1>${wheel_mu}</mu1>
-        <mu2>${wheel_mu}</mu2>
+    <!--<gazebo reference="front_left_wheel">
+        <mu1>${wheel_mu1}</mu1>
+        <mu2>${wheel_mu2}</mu2>
     </gazebo>
     <gazebo reference="front_right_wheel">
-        <mu1>${wheel_mu}</mu1>
-        <mu2>${wheel_mu}</mu2>
+        <mu1>${wheel_mu1}</mu1>
+        <mu2>${wheel_mu2}</mu2>
     </gazebo>
     <gazebo reference="rear_left_wheel">
-        <mu1>${wheel_mu}</mu1>
-        <mu2>${wheel_mu}</mu2>
+        <mu1>${wheel_mu1}</mu1>
+        <mu2>${wheel_mu2}</mu2>
     </gazebo>
     <gazebo reference="rear_right_wheel">
-        <mu1>${wheel_mu}</mu1>
-        <mu2>${wheel_mu}</mu2>
-    </gazebo>
+        <mu1>${wheel_mu1}</mu1>
+        <mu2>${wheel_mu2}</mu2>
+    </gazebo>-->
     <!-- design transmission for joint-->
-    <joint_trans joint_name="front_right_wheel_joint"/>
+    <!--<joint_trans joint_name="front_right_wheel_joint"/>
     <joint_trans joint_name="front_left_wheel_joint"/>
-    <!--<joint_trans joint_name="rear_right_wheel_joint"/>
+    <joint_trans joint_name="rear_right_wheel_joint"/>
     <joint_trans joint_name="rear_left_wheel_joint"/>-->
-    <!--<joint_trans joint_name="paddle_joint"/>-->
+    <joint_trans joint_name="paddle_joint"/>
     <gazebo>
-        <plugin name="differential_drive_controller" filename="libgazebo_ros_diff_drive.so">
-            <rosDebugLevel>Debug</rosDebugLevel>
-            <publishWheelTF>true</publishWheelTF>
+        <plugin name="skid_steer_drive_controller" filename="libgazebo_ros_skid_steer_drive.so">
+            <updateRate>50.0</updateRate>
             <robotNamespace>/</robotNamespace>
-            <publishTf>1</publishTf>
-            <publishWheelJointState>true</publishWheelJointState>
-            <alwaysOn>true</alwaysOn>
-            <updateRate>100.0</updateRate>
-            <legacyMode>true</legacyMode>
-            <leftJoint>front_left_wheel_joint</leftJoint>
-            <rightJoint>front_right_wheel_joint</rightJoint>
+            <leftFrontJoint>front_left_wheel_joint</leftFrontJoint>
+            <leftRearJoint>rear_left_wheel_joint</leftRearJoint>
+            <rightFrontJoint>front_right_wheel_joint</rightFrontJoint>
+            <rightRearJoint>rear_right_wheel_joint</rightRearJoint>
             <wheelSeparation>0.12</wheelSeparation>
             <wheelDiameter>0.064</wheelDiameter>
-            <broadcastTF>1</broadcastTF>
-            <wheelTorque>30</wheelTorque>
-            <wheelAcceleration>1.8</wheelAcceleration>
-            <commandTopic>cmd_vel</commandTopic>
-            <odometryFrame>odom</odometryFrame>
+            <commandTopic>/cmd_vel</commandTopic>
             <odometryTopic>odom</odometryTopic>
             <robotBaseFrame>base_footprint</robotBaseFrame>
+            <odometryFrame>odom</odometryFrame>
+            <torque>1</torque>
+            <topicName>/cmd_vel</topicName>
+            <broadcastTF>1</broadcastTF>
         </plugin>
     </gazebo>
-    <!-- design controller for joint-->
-    <!--<gazebo>
-        <plugin name="gazebo_ros_control" filename="libgazebo_ros_control.so">
-            <robotNamespace>/pick_ball_mbot</robotNamespace>
-            <robotSimType>gazebo_ros_control/DefaultRobotHWSim</robotSimType>
-            <legacyModeNS>true</legacyModeNS>
-            </plugin>
-    </gazebo>-->
 </robot>

File: src/pick_ball_mbot/pick_ball_mbot_description/urdf/sensors/kinect_gazebo.xacro (robot description, xacro)
@@ -9,10 +9,10 @@
                 <origin xyz="0 0 0" rpy="0 0 ${M_PI/2}"/>
                 <geometry>
-                    <mesh scale="0.5 0.5 0.5" filename="package://pick_ball_mbot_description/meshes/kinect.dae" />
+                    <mesh scale="0.25 0.25 0.25" filename="package://pick_ball_mbot_description/meshes/kinect.dae" />
                 </geometry>
             </visual>
             <collision>
                 <geometry>
-                    <box size="0.035 0.15 0.045" />
+                    <box size="0.017 0.07 0.022" />
                 </geometry>
             </collision>
@@ -29,5 +29,5 @@
                 <update_rate>20.0</update_rate>
                 <camera>
-                    <horizontal_fov>${90.0*M_PI/180.0}</horizontal_fov>
+                    <horizontal_fov>${60*M_PI/180.0}</horizontal_fov>
                     <image>
                         <format>R8G8B8</format>
@@ -37,5 +37,5 @@
                     <clip>
                         <near>0.05</near>
-                        <far>8.0</far>
+                        <far>8</far>
                     </clip>
                 </camera>

File: src/pick_ball_mbot/pick_ball_mbot_description/urdf/sensors/lidar_gazebo.xacro (robot description, xacro)
@@ -14,5 +14,5 @@
                 <origin xyz=" 0 0 0 " rpy="0 0 0" />
                 <geometry>
-                    <cylinder length="0.025" radius="0.025"/>
+                    <cylinder length="0.02" radius="0.02"/>
                 </geometry>
                 <material name="black"/>
@@ -21,5 +21,5 @@
                 <origin xyz="0.0 0.0 0.0" rpy="0 0 0" />
                 <geometry>
-                    <cylinder length="0.03" radius="0.025"/>
+                    <cylinder length="0.02" radius="0.02"/>
                 </geometry>
             </collision>
